File: PWM3360 Breakout Board.kicad_pcb (KiCad board)
At the start: 2 copper layers, 29.5 x 32.5 mm, 11 parts, among them J1 Conn_01x06, J2 Conn_01x06, U1 PMW3360, U2 TLV70019_SOT23-5

Commit message: make it more smaller
Routing:
- net GND: track 59.6 -> 62.3 mm
- net MISO: track 45.2 -> 44.1 mm
- net NCS: track 25.3 -> 24.5 mm
Other:
- board size 29.5 x 32.5 mm -> 29.5 x 31.5 mm
- board text added: "PMW3360 Breakout Board V1 14/08/2022"
- board text removed: "PMW3360 Breakout Board V1 14/08/2022 https://github.com/karnadii/ pwm3360_breakout_board"
