File: _autosave-PWM3360 Breakout Board.kicad_pcb (KiCad board)
At the start: 2 copper layers, 29.5 x 32.5 mm, 11 parts, among them J1 Conn_01x06, J2 Conn_01x06, U1 PMW3360, U2 TLV70019_SOT23-5

Commit message: make it more smaller
Parts:
- moved J1 0.83 mm to (129.5, 87.7)
- moved J2 0.83 mm to (135.9, 87.5)
Routing:
- net NCS: track 25.3 -> 17.0 mm
- net MISO: track 45.2 -> 37.8 mm
- net MOSI: track 36.6 -> 31.6 mm
- net GND: track 59.6 -> 64.2 mm
- net SCLK: track 43.4 -> 40.4 mm
- net +3V3: track 49.3 -> 50.2 mm
Other:
- board size 29.5 x 32.5 mm -> 29.5 x 30.8 mm
- board text added: "PMW3360 Breakout Board V1 14/08/2022"
- board text removed: "PMW3360 Breakout Board V1 14/08/2022 https://github.com/karnadii/ pwm3360_breakout_board"

Commit message: add readme
Other:
- board text added: "GND CS MOSI 3V3 MISO CLK"
- board text removed: "GND|3V3|CS|MISO|MOSI|CLK"
Changed lines of the file:
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@@
   (gr_line (start 119.425 101.67) (end 121.925 108.67) (layer "Edge.Cuts") (width 0.1))
   (gr_line (start 129.425 83.17) (end 135.675 83.17) (layer "Edge.Cuts") (width 0.1))
-  (gr_text "GND|3V3|CS|MISO|MOSI|CLK" (at 129.425 84.42) (layer "B.SilkS")
-    (effects (font (size 0.8 0.8) (thickness 0.15)) (justify mirror))
+  (gr_text "GND  \n\nCS \n\nMOSI\n\n3V3 \n\nMISO\n\nCLK" (at 129.425 86.42 270) (layer "B.SilkS")
+    (effects (font (size 0.8 0.8) (thickness 0.15)) (justify left mirror))
   )
   (gr_text "PMW3360 Breakout \nBoard V1\n14/08/2022\n\n" (at 129.425 110.92) (layer "B.SilkS")
